File: FuzzFace2/FuzzFace2copy.kicad_pcb (KiCad board)
At the start: 2 copper layers, 54 x 62 mm, 22 parts, among them Q1 2SA1015, Q2 2SA1015

Commit message: fuzz face v2 files
Parts:
- added H10: In GND, ANA PARTS:1.5mm_MountingHole, F.Cu at (144.2, 81.2)
- added H11: Out GND, ANA PARTS:1.5mm_MountingHole, F.Cu at (171.2, 81.2)
- H4: value +9V -> GND
- moved H3 4.76 mm to (139.2, 81.2)
- moved C1 0.35 mm to (142.5, 74.2)
- moved C2 0.35 mm to (132.5, 58.2)
- moved C3 0.35 mm to (173.2, 58.8)
- moved D1 0.35 mm to (146.5, 74.2)
- moved H1 0.35 mm to (149.2, 81.2)
- moved H2 0.35 mm to (166.2, 81.2)
- moved H4 0.35 mm to (154.2, 81.2)
- moved H5 0.35 mm to (161.2, 81.2)
- moved H6 0.35 mm to (131.2, 31.2)
- moved H7 0.35 mm to (179.2, 31.2)
- moved H8 0.35 mm to (131.2, 86.2)
- moved H9 0.35 mm to (179.2, 86.2)
- moved Q1 0.35 mm to (141.0, 62.4)
- moved Q2 0.35 mm to (147.0, 63.2)
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Connections:
- H4 pad 1: Net-(H4-Pad1) -> GND
- R5 pad 1: Net-(H4-Pad1) -> GND
Routing:
- net Net-(H4-Pad1): track 8.09 -> 0.00 mm
- net GND: track 10.3 -> 18.4 mm
- net Net-(D1-K): track 7.68 -> 10.1 mm
