File: FuzzFace2/FuzzFace2copy.kicad_sch (KiCad schematic)
At the start: 22 parts, among them Q1 2SA1015, Q2 2SA1015

Commit message: fuzz face v2 files
Parts:
- added H10: In GND, ANA PARTS:1.5mm_MountingHole, symbol Mechanical:MountingHole_Pad
- added H11: Out GND, ANA PARTS:1.5mm_MountingHole, symbol Mechanical:MountingHole_Pad
- H4: value +9V -> GND
Connections:
- net GND: now also H4.1, R5.1, H10.1, H11.1
Other:
- moved on the sheet: H6, H7, H8, H9
