File: FuzzFaceV3/REALFUZZFACE.kicad_sch (KiCad schematic)
At the start: 24 parts, among them Q1 2SA1015, Q2 2SA1015

Commit message: done
Parts:
- removed H9: MountingHole, MountingHole:MountingHole_2.2mm_M2_DIN965_Pad_TopOnly, symbol Mechanical:MountingHole
- IN: renamed from H1; value Input -> IN
- IN_GND: renamed from H10; value In GND -> IN_GND
- MH1: renamed from H6; value MountingHole -> MH1
- MH2: renamed from H7; value MountingHole -> MH2
- OUT: renamed from H2; value Output -> OUT
- OUT_GND: renamed from H11; value Out GND -> OUT_GND
- PWR: renamed from H5; value -9V -> PWR
- P_GND: renamed from H8; value MountingHole -> P_GND
- renumbered C1 to C?, C2 to C?, C3 to C?, D1 to D?, H4 to GND, Q1 to Q?, Q2 to Q?, R2 to R?, R5 to R?, R1 to R?, R4 to R?, R3 to R?, R_fuzz1 to R_fuzz?, R_vol1 to R_vol?, H3 to SW
